File: Entwicklung_Leiterplatte/Leiterplatte_Steuerbox.kicad_pcb (KiCad board)
At the start: 2 copper layers, 169.8 x 56.3 mm, 33 parts, among them U1 ESP32-S3-ETH, U2 ESP32-DevKitC

Commit message: Improved traces + improved silkscreen
Routing:
- net /SDA_ESP32ETH: track 106.5 -> 105.4 mm
- net /SCL_ESP32ETH: track 100.0 -> 99.0 mm
Other:
- board text added: "24V"
- board text added: "3V3"
- board text added: "5V"
- board text added: "9V"
- board text added: "A+"
- board text added: "A-"
- board text added: "B+"
- board text added: "B-"
- board text added: "DIR"
- board text added: "EN"
- board text added: "GND"
- board text added: "SCL"
- board text added: "SDA"
- board text added: "SIG"
- board text added: "STP"
- board text added: "XSHUT"
